Commit message: updata code

File: environment_description/simulation_table/object3.urdf (robot description, URDF)
Before this commit: robot objects, 2 links, 1 joints
Links:
- link cylinder1: geometry collision mesh filename=meshes/square.stl; visual mesh filename=meshes/square.stl

File: environment_description/simulation_table/object4.urdf (robot description, URDF)
Before this commit: robot objects, 2 links, 1 joints
Links:
- link cylinder1: geometry collision mesh filename=meshes/square.stl; visual mesh filename=meshes/square.stl

File: environment_description/simulation_table/object5.urdf (robot description, URDF)
Before this commit: robot objects, 2 links, 1 joints
Links:
- removed link table
- added link cylinder1, mass 0.5; collision mesh filename=meshes/square.stl; visual mesh filename=meshes/square.stl
Joints:
- removed joint table_link_to_world
- added joint cylinder1_to_world: type floating, parent World, child cylinder1, origin xyz=0. 0. 0. rpy=0.0 0.0 0.0

File: environment_description/simulation_table/object6.urdf (robot description, URDF)
Before this commit: robot objects, 2 links, 1 joints
Links:
- link cylinder1: geometry collision mesh filename=meshes/triangle.stl; visual mesh filename=meshes/triangle.stl

File: environment_description/simulation_table/object7.urdf (robot description, URDF)
Before this commit: robot objects, 2 links, 1 joints
Links:
- link cylinder1: geometry collision mesh filename=meshes/triangle.stl; visual mesh filename=meshes/triangle.stl

File: environment_description/simulation_table/object8.urdf (robot description, URDF)
Before this commit: robot objects, 2 links, 1 joints
Links:
- link cylinder1: geometry collision mesh filename=meshes/triangle.stl; visual mesh filename=meshes/triangle.stl
